Commit message: updated maara and zivid urdfs so that zivid urdfs are as per original copied from pull request made to official zivid-ros repo except that collision object is scaled up and collision origin is moved to accomodate that. Cable urdf is now in maara_joint_limited_ur5. Transforms for zivid links relative to ur5 are now in maara_joint_limited_ur5.

File: zivid_description/urdf/macros/zivid_camera.xacro (robot description, xacro)
@@ -8,15 +8,17 @@
             <!-- Visuals -->
             <visual>
-                <origin xyz="0.057 -0.1095 -0.074" rpy="${0.5*M_PI} ${-0.5*M_PI} ${0.5*M_PI}"/> <!--0.057 -0.1045 -0.074--> <!--"-0.0030 -0.0758 0.0445"-->
+                <!--origin xyz="0.057 -0.1095 -0.074" rpy="${0.5*M_PI} ${-0.5*M_PI} ${0.5*M_PI}"/--> <!--0.057 -0.1045 -0.074--> <!--"-0.0030 -0.0758 0.0445"-->
+				 <origin xyz="-0.0030 -0.0758 0.0445" rpy="${0.5*M_PI} 0 ${0.5*M_PI}"/>
                 <material name="blue">
                     <color rgba="0.25 0.25 0.25 1"/>
                 </material>
                 <geometry>
-                    <mesh filename="package://zivid_description/meshes/visual/zivid-one-plus.stl" scale="0.0011 0.0011 0.0011"/>
+                    <mesh filename="package://zivid_description/meshes/visual/zivid-one-plus.stl" scale="0.001 0.001 0.001"/>
                 </geometry>
             </visual>
             <!-- Collisions -->
             <collision>
-                <origin xyz="0.057 -0.1095 -0.074" rpy="${0.5*M_PI} ${-0.5*M_PI} ${0.5*M_PI}"/> <!--xyz="0.057 -0.1045 -0.074"-->
+                <!--origin xyz="0.057 -0.1095 -0.074" rpy="${0.5*M_PI} ${-0.5*M_PI} ${0.5*M_PI}"/--> <!--xyz="0.057 -0.1045 -0.074"-->
+                <origin xyz="-0.0043 -0.083 0.0483" rpy="${0.5*M_PI} 0 ${0.5*M_PI}"/>
                 <geometry>
                     <mesh filename="package://zivid_description/meshes/collision/zivid-one-plus.stl" scale="0.0011 0.0011 0.0011"/>
@@ -24,27 +26,4 @@
             </collision>
         </link>
-		<joint name="${prefix}cables_joint" type="fixed">
-            <origin xyz="0 0 0" rpy="0 0 0"/>
-            <parent link="${prefix}base_link"/>
-            <child link="${prefix}cables_link"/>
-        </joint>
-		<link name="${prefix}cables_link">
-		<visual>
-			<material name="blue">
-                <color rgba="0.25 0.25 0.25 1"/>
-            </material>
-			<geometry>
-                <box size="0.04 0.02 0.08"/> <!--"0.08 0.04 0.08"-->
-            </geometry>
-				<origin xyz="-0.05 -0.115 0.025" rpy="0 0 0"/> <!--xyz="-0.035 -0.115 0.025"--> <!--"-0.032 -0.11 0.02"-->
-        </visual>
-        <!-- Collisions -->
-        <collision>
-            <geometry>
-                <box size="0.04 0.02 0.08"/>
-            </geometry>
-				<origin xyz="-0.05 -0.115 0.025" rpy="0 0 0"/>
-        </collision>
-		</link>
         <!-- Zivid Optical (Measurement) and Projector Frames -->
         <link name="${prefix}optical_frame"/>

Commit message: update zivid-ros sampling and urdf

File: zivid_description/urdf/macros/zivid_camera.xacro (robot description, xacro)
@@ -9,5 +9,6 @@
             <visual>
                 <!--origin xyz="0.057 -0.1095 -0.074" rpy="${0.5*M_PI} ${-0.5*M_PI} ${0.5*M_PI}"/--> <!--0.057 -0.1045 -0.074--> <!--"-0.0030 -0.0758 0.0445"-->
-				 <origin xyz="-0.0030 -0.0758 0.0445" rpy="${0.5*M_PI} 0 ${0.5*M_PI}"/>
+				<origin xyz="-0.0030 -0.0758 0.0445" rpy="${0.5*M_PI} 0 ${0.5*M_PI}"/>
+				<!-- <origin xyz="-0.0043 -0.083 0.0483" rpy="${0.5*M_PI} 0 ${0.5*M_PI}"/> -->
                 <material name="blue">
                     <color rgba="0.25 0.25 0.25 1"/>
@@ -32,4 +33,5 @@
         <joint name="${prefix}optical_joint" type="fixed">
             <origin xyz="0.065 0.062 0.0445" rpy="-${0.5*M_PI} 0 -${0.5*M_PI + 8.5/180*M_PI}"/>
+            <!-- <origin xyz="${0.065*1.1} ${0.062*1.1} ${0.0445*1.1}" rpy="-${0.5*M_PI} 0 -${0.5*M_PI + 8.5/180*M_PI}"/> -->
             <parent link="${prefix}base_link"/>
             <child link="${prefix}optical_frame"/>
@@ -37,4 +39,5 @@
         <joint name="${prefix}projector_joint" type="fixed">
             <origin xyz="-0.0030 -0.0758 0.0445" rpy="-${0.5*M_PI} 0 -${0.5*M_PI}"/>
+            <!-- <origin xyz="${-0.0030*1.1} ${-0.0758*1.1} ${0.0445*1.1}" rpy="-${0.5*M_PI} 0 -${0.5*M_PI}"/> -->
             <parent link="${prefix}base_link"/>
             <child link="${prefix}projector_frame"/>

Commit message: urdf + bringup

File: zivid_description/urdf/macros/zivid_camera.xacro (robot description, xacro)
@@ -31,10 +31,9 @@
         <link name="${prefix}projector_frame"/>
         <!-- Zivid Optical (Measurement) and Projector Joints -->
-        <joint name="${prefix}optical_joint" type="fixed">
+        <!--<joint name="${prefix}optical_joint" type="fixed">
             <origin xyz="0.065 0.062 0.0445" rpy="-${0.5*M_PI} 0 -${0.5*M_PI + 8.5/180*M_PI}"/>
-            <!-- <origin xyz="${0.065*1.1} ${0.062*1.1} ${0.0445*1.1}" rpy="-${0.5*M_PI} 0 -${0.5*M_PI + 8.5/180*M_PI}"/> -->
             <parent link="${prefix}base_link"/>
             <child link="${prefix}optical_frame"/>
-        </joint>
+        </joint>-->
         <joint name="${prefix}projector_joint" type="fixed">
             <origin xyz="-0.0030 -0.0758 0.0445" rpy="-${0.5*M_PI} 0 -${0.5*M_PI}"/>
